File: hardware/PelletMon.kicad_pcb (KiCad board)
At the start: 4 copper layers, 48 x 31.4 mm, 18 parts, among them J1 USB_B_Micro, J2 Conn_01x03, J3 Conn_01x04, J4 Conn_01x02, U1 SN65HVD230, U2 AMS1117-3.3, U3 ESP32-WROOM-32

Commit message: PCB update
Routing:
- net /USS_TRIG: track 46.9 -> 58.2 mm
- net GND: vias 22 -> 19
- net +3V3: vias 9 -> 11
Other:
- rule via_min_size: 0.4 -> 0.5
- board text added: "use rx+tx to upload"
- board text removed: "use rx/tx to upload"

Commit message: Update gerbers and renders
Routing:
- net Net-(J1-Pad6): track 0.00 -> 12.1 mm
- net +3V3: track 7.57 -> 7.31 mm, vias 11 -> 10
- net GND: vias 19 -> 20
- removed copper zone on F.Cu, net Net-(J1-Pad6)
