File: hardware/PelletMon.kicad_pcb (KiCad board)
At the start: 4 copper layers, 48 x 31.4 mm, 18 parts, among them J1 USB_B_Micro, J2 Conn_01x03, J3 Conn_01x04, J4 Conn_01x02, U1 SN65HVD230, U2 AMS1117-3.3, U3 ESP32-WROOM-32

Commit message: Last fixes before fab
Routing:
- net GND: vias 20 -> 21

Commit message: Before FAB
Routing:
- net GND: vias 21 -> 24

Commit message: Minor PCB tweaks
Connections:
- net Net-(J4-Pad1) renamed /CAN_P
- net Net-(J4-Pad2) renamed /CAN_N
Routing:
- net /USS_TRIG: track 58.2 -> 43.6 mm
- net /CAN_N: track 8.75 -> 10.1 mm
- net Net-(C4-Pad1): track 8.17 -> 7.48 mm
- net /CAN_P: track 9.46 -> 10.1 mm
- net +3V3: track 7.31 -> 6.73 mm
Other:
- net class CAN added: clearance 0.2, trace_width 0.32, via_dia 0.6, via_drill 0.3
- net class PWR added: clearance 0.2, trace_width 0.9, via_dia 0.6, via_drill 0.3

Commit message: Misc tweaks
Other:
- net class CAN: trace_width 0.32 -> 0.2
- net class Default: trace_width 0.25 -> 0.35
