File: hardware/PelletMon.sch (KiCad schematic (older format))
At the start: 18 parts, among them J1 USB_B_Micro, J2 Conn_01x03, J3 Conn_01x04, J4 Conn_01x02, U1 SN65HVD230, U2 AMS1117-3.3, U3 ESP32-WROOM-32

Commit message: Minor PCB tweaks
Connections:
- net CAN_N: now reaches J4.2 (Pin_2), R9.2, U1.6 (CANL)
- net CAN_P: now reaches J4.1 (Pin_1), R9.1, U1.7 (CANH)
Changed lines of the file:
@@
 NoConn ~ 7275 3450
 NoConn ~ 3225 3025
+Text Label 4250 4125 0    50   ~ 0
+CAN_P
+Text Label 4250 4525 0    50   ~ 0
+CAN_N
 $EndSCHEMATC
